File: Pro/PCB/Lily58_Pro.kicad_pcb (KiCad board)
At the start: 2 copper layers, 142.5 x 106.3 mm, 87 parts, among them J1 LED, J2 4PIN, J3 OLED, P1 i2c_pin, P2 i2c_pin, SW1 SW_PUSH, SW10 SW_PUSH, SW11 SW_PUSH, SW12 SW_PUSH, SW13 SW_PUSH, SW14 SW_PUSH, SW15 SW_PUSH, SW16 SW_PUSH, SW17 SW_PUSH, SW18 SW_PUSH, SW19 SW_PUSH, SW2 SW_PUSH, SW20 SW_PUSH, SW21 SW_PUSH, SW22 SW_PUSH, SW23 SW_PUSH, SW24 SW_PUSH, SW25 SW_PUSH, SW26 SW_PUSH, SW27 SW_PUSH, SW28 SW_PUSH, SW29 SW_PUSH, SW3 SW_PUSH, SW4 SW_PUSH, SW5 SW_PUSH, SW6 SW_PUSH, SW7 SW_PUSH, SW8 SW_PUSH, SW9 SW_PUSH, U1 ProMicro

Commit message: palm key and stagger modifications to pcb
Parts:
- removed G*** (x2): LOGO, Lily58-footprint:lily58_logo_2
- removed G*** (x2): LOGO, Lily58-footprint:lily58_logo_Pro
- added TH3: HOLE, Lily58-footprint:HOLE_M2_TH, F.Cu at (127.5, 158.5)
- JP1, JP2, JP3, JP4, JP5, JP6, JP7, JP8: value (none) -> Jumper_NO_Small
- SW1, SW10, SW11, SW12, SW13, SW14, SW15, SW16, SW17, SW18, SW19, SW2, SW20, SW21, SW22, SW23, SW24, SW25, SW26, SW27, SW28, SW29, SW3, SW4, SW5, SW6, SW7, SW8, SW9: footprint Lily58-footprint:CherryMX_KailhLowProfile_Hotswap_edge -> Lily58-footprint:CherryMX_KailhLowProfile_Hotswap
- moved SW29 67.1 mm to (132.1, 180.3)
- moved D29 61.6 mm to (137.7, 172.5), turned to 180 degrees
- moved D24 1.05 mm to (221.6, 104.1)
- moved D6 1.05 mm to (221.5, 62.8)
- moved D11 1.05 mm to (190.3, 64.3)
- moved D17 1.05 mm to (190.3, 99.3)
- moved D23 1.05 mm to (190.3, 102.5)
- moved SW11 1.05 mm to (196.4, 72.3)
- moved SW12 1.05 mm to (215.4, 73.8)
- moved SW17 1.05 mm to (196.4, 91.5)
- moved SW18 1.05 mm to (215.4, 93.0)
- moved SW23 1.05 mm to (196.4, 110.5)
- moved SW24 1.05 mm to (215.5, 112.0)
- moved D12 1.05 mm to (221.5, 65.9)
- moved D18 1.05 mm to (221.5, 100.9)
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Routing:
- net col1: track 350.6 -> 436.2 mm
- net row4: track 132.6 -> 206.5 mm
- net col2: track 334.4 -> 323.5 mm
- net Net-(D29-Pad2): track 36.9 -> 28.3 mm, vias 2 -> 1
- net col0: track 304.4 -> 300.8 mm
- net Net-(D24-Pad2): track 28.1 -> 31.4 mm, vias 2 -> 1
- net Net-(D12-Pad2): track 28.0 -> 30.6 mm, vias 2 -> 1
- net row2: track 165.8 -> 167.5 mm
- net Net-(D23-Pad2): track 37.1 -> 35.4 mm
- net Net-(D9-Pad2): track 36.9 -> 35.4 mm
- net Net-(D7-Pad2): track 37.3 -> 35.7 mm
- net Net-(D4-Pad2): track 28.0 -> 26.5 mm
- net Net-(D3-Pad2): track 28.0 -> 26.5 mm
- net Net-(D28-Pad2): track 37.1 -> 35.5 mm
- net Net-(D27-Pad2): track 37.1 -> 35.5 mm
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Other:
- board size 142.5 x 106.3 mm -> 142.3 x 153.4 mm
